File: MonT_Feather.kicad_pcb (KiCad board)
At the start: 2 copper layers, 50.8 x 22.9 mm, 11 parts, among them J1 Adafruit_Feather, J2 DB25_Male, U1 MAX3232

Commit message: DSR_TTL pulldown
Parts:
- added R1: 15k, 0_LOCAL:R_0805, F.Cu at (140.0, 103.2)
- moved JP1 4.66 mm to (127.5, 90.4)
Routing:
- net /RTS: track 45.6 -> 46.1 mm

Commit message: alternate routing
Parts:
- moved C4 1.35 mm to (155.3, 92.0), turned to 0 degrees
- moved C3 1.20 mm to (155.3, 95.6), turned to 0 degrees
Routing:
- net /RTS: track 46.1 -> 31.7 mm
- net /CTS: track 37.8 -> 28.7 mm
- net /RXD: track 11.9 -> 13.1 mm, vias 1 -> 0
- net /TXD: track 17.4 -> 17.5 mm, vias 1 -> 0
- net +3V3: vias 0 -> 1
