File: MounT_Feather.sch (KiCad schematic (older format))
At the start: 11 parts, among them J1 Adafruit_Feather, J2 DB25_Male, U1 MAX3232

Commit message: reduce pin stagger offset to 4mil
Parts:
- J1: footprint 0_LOCAL:Adafruit_Feather_stagger -> 0_LOCAL:Adafruit_Feather_stagger_4mil
Changed lines of the file:
@@
 F 0 "J1" H 2490 4380 60  0000 L CNN
 F 1 "Adafruit_Feather" V 2760 3930 60  0000 L CNN
-F 2 "0_LOCAL:Adafruit_Feather_stagger" H 925 2285 60  0001 L CNN
+F 2 "0_LOCAL:Adafruit_Feather_stagger_4mil" H 925 2285 60  0001 L CNN
 F 3 "http://ww1.microchip.com/downloads/en/DeviceDoc/Atmel-7766-8-bit-AVR-ATmega16U4-32U4_Summary.pdf" H 925 2385 60  0001 L CNN
 F 4 "Active" H 2750 5460 60  0001 L CNN "Status"

Commit message: use 6mil stagger, 4mil wasn't good enough
Parts:
- J1: footprint 0_LOCAL:Adafruit_Feather_stagger_4mil -> 0_LOCAL:Adafruit_Feather_stagger_6mil
Changed lines of the file:
@@
 F 0 "J1" H 2490 4380 60  0000 L CNN
 F 1 "Adafruit_Feather" V 2760 3930 60  0000 L CNN
-F 2 "0_LOCAL:Adafruit_Feather_stagger_4mil" H 925 2285 60  0001 L CNN
+F 2 "0_LOCAL:Adafruit_Feather_stagger_6mil" H 925 2285 60  0001 L CNN
 F 3 "http://ww1.microchip.com/downloads/en/DeviceDoc/Atmel-7766-8-bit-AVR-ATmega16U4-32U4_Summary.pdf" H 925 2385 60  0001 L CNN
 F 4 "Active" H 2750 5460 60  0001 L CNN "Status"
