File: MounT_Teensy.kicad_pcb (KiCad board)
At the start: 2 copper layers, 61.2 x 18 mm, 10 parts, among them J1 Teensy, J2 DB25_Male, U1 MAX3232

Commit message: nothing really
Parts:
- NT1: footprint 0_LOCAL:NetTie-2_SMD_10 -> 0_LOCAL:NetTie-2_SMD_0.2
- moved C5 2.13 mm to (171.4, 100.7), turned to 0 degrees
- moved C2 0.33 mm to (171.4, 98.8)
- moved J2 0.05 mm to (163.9, 95.1)
- moved NT1 0.05 mm to (147.3, 96.5)
Routing:
- net +3V3: track 11.4 -> 12.5 mm
- net /CTS_232: track 39.1 -> 38.4 mm
Other:
- net class Default: clearance 0.1778 -> 0.2; trace_width 0.1778 -> 0.2; via_dia 0.4064 -> 0.5; via_drill 0.254 -> 0.3
- rule trace_clearance: 0.1778 -> 0.2
- rule trace_min: 0.1778 -> 0.2
- rule via_min_drill: 0.254 -> 0.3
- rule via_min_size: 0.4064 -> 0.5
- board text added: "v003"
