File: MounT_Feather.kicad_pcb (KiCad board)
At the start: 2 copper layers, 50.8 x 22.9 mm, 11 parts, among them J1 Adafruit_Feather, J2 DB25_Male, U1 MAX3232

Commit message: nothing really
Parts:
- NT1: footprint 0_LOCAL:NetTie-2_SMD_10 -> 0_LOCAL:NetTie-2_SMD_0.2
Routing:
- net /TX_232: track 16.8 -> 17.7 mm
- net /TX_TTL: track 20.1 -> 19.2 mm
- net /RX_TTL: track 18.7 -> 18.0 mm
- net /En: track 19.7 -> 19.1 mm
- net /RTS_232: track 47.6 -> 47.0 mm
- net GND: vias 0 -> 4
Other:
- net class Default: clearance 0.1778 -> 0.2; trace_width 0.1778 -> 0.2; via_dia 0.4064 -> 0.5; via_drill 0.254 -> 0.3
- rule trace_clearance: 0.1778 -> 0.2
- rule trace_min: 0.1778 -> 0.2
- rule via_min_drill: 0.254 -> 0.3
- rule via_min_size: 0.4064 -> 0.5
- board text added: "v003"
- board text removed: "Feather"
- board text removed: "MounT"

Commit message: mostly just readme & link to pcbway
Parts:
- NT1: moved to B.Cu
Routing:
- net /DTR_232: track 13.1 -> 11.7 mm
- net /TX_232: track 17.7 -> 16.9 mm
- net GND: vias 4 -> 0
Other:
- board text added: "Use ENIG finish. DIP holes are a connector."
- board text added: "github.com/bkw777/MounT - v004"
- board text removed: "github.com/bkw777/MounT"
- board text removed: "v003"
