File: MounT_Feather_WP-2.kicad_pcb (KiCad board)
At the start: 2 copper layers, 50.8 x 22.9 mm, 11 parts, among them J1 Adafruit_Feather, J2 DE9_Female, U1 MAX3232

Commit message: mostly just readme & link to pcbway
Routing:
- net /CTS_232: track 35.0 -> 32.8 mm
- net /DSR_232: track 12.7 -> 14.6 mm
- net /RX_TTL: track 18.7 -> 17.8 mm
- net /DSR_TTL: track 14.4 -> 15.3 mm
- net /TX_TTL: track 19.9 -> 19.1 mm
- net /En: track 19.8 -> 19.1 mm
- net /DTR_232: track 13.5 -> 12.8 mm
- net /RTS_232: track 24.0 -> 23.5 mm
