File: MounT_K85_Teensy.kicad_pcb (KiCad board)
At the start: 2 copper layers, 61.2 x 18 mm, 9 parts, among them J1 Teensy_3.5_3.6_4.1_DIP_only, J2 DB25_Male, U1 MAX3232

Commit message: smt power switch on feather, routing 3v3 on teensy, silkscreen all
Parts:
- J1: value Teensy_3.5_3.6_4.1_DIP_only -> Teensy_3.5_3.6_4.1
Routing:
- net +3V3: track 48.7 -> 48.2 mm, vias 5 -> 3
- net GND: vias 8 -> 2
